File: PCB/SLIDER_PCB_REV_A/SLIDER_PCB_REV_A.kicad_sch (KiCad schematic)
At the start: 5 parts, among them J1 V0, SW1 SW_Push

Commit message: 21h30 update : cad and PCB changes
Parts:
- removed SW1: SW_Push, Connector_PinHeader_2.54mm:PinHeader_1x02_P2.54mm_Vertical, symbol Switch:SW_Push
- added C2: C_Polarized, Capacitor_THT:C_Disc_D5.0mm_W2.5mm_P5.00mm, symbol Device:C_Polarized
- added J2, J3: V0, Connector_PinHeader_2.54mm:PinHeader_1x04_P2.54mm_Vertical, symbol Connector:Conn_01x04_Pin
- added J4, J5: Conn_01x02_Pin, Connector_PinHeader_2.54mm:PinHeader_1x02_P2.54mm_Vertical, symbol Connector:Conn_01x02_Pin
- A1, A2: footprint Module:Pololu_Breakout-16_15.2x20.3mm -> ESP32-S3:Pololu_Breakout-16_15.2x20.3mm
- J1: footprint (none) -> Connector_PinHeader_2.54mm:PinHeader_1x04_P2.54mm_Vertical
Connections:
- net GND: now reaches A2.1 (GND)
- net GND: now also A1.1 (GND), A1.7 (GND), A2.7 (GND), ESP32_S1.4 (GND), J1.2 (GND), C2.2, J4.2 (Pin_2), J5.2 (Pin_2)
- net VDD: now reaches A2.10 (MS1)
- net VDD: now also A1.10 (MS1), A1.11 (MS2), A1.12 (MS3), A1.2 (VDD), A2.11 (MS2), A2.12 (MS3), A2.2 (VDD), ESP32_S1.2 (5V), J1.1 (V0)
- net at A2.13 (~{RESET}): now also A2.14 (~{SLEEP})
- net at A2.15 (STEP): now also ESP32_S1.13 (5)
- net at A2.16 (DIR): now also ESP32_S1.11 (4)
- net at A2.3 (1B): now also J3.4 (EN)
- net at A2.4 (1A): now also J3.3 (IN+)
- net at A2.5 (2A): now also J3.2 (GND)
- net at A2.6 (2B): now also J3.1 (V0)
- net +12V: now reaches A2.8 (VMOT)
- net +12V: now also A1.8 (VMOT), J1.3 (IN+), C2.1, J4.1 (Pin_1)
- net at A2.9 (~{ENABLE}): now also ESP32_S1.15 (6)
- net at A1.13 (~{RESET}): now also A1.14 (~{SLEEP})
- net at A1.15 (STEP): now also ESP32_S1.7 (2)
- net at A1.16 (DIR): now also ESP32_S1.5 (1)
- net at A1.3 (1B): now also J2.4 (EN)
- net at A1.4 (1A): now also J2.3 (IN+)
- net at A1.5 (2A): now also J2.2 (GND)
- net at A1.6 (2B): now also J2.1 (V0)
- net at A1.9 (~{ENABLE}): now also ESP32_S1.9 (3)
- new net: ESP32_S1.8 (13), J5.1 (Pin_1)
- no-connect marks 0 -> 20
Other:
- moved on the sheet: A1, A2, J1
