File: PCB/CONTROLLER_PCB_REV_A/controller/controller.kicad_sch (KiCad schematic)
At the start: 10 parts, among them J1 Conn_01x05_Pin, J2 Conn_01x05_Pin, J3 Conn_01x09_Pin, J6 Conn_01x04_Pin, J7 Conn_01x04_Pin, U2 MCP23017_SP

Commit message: Added 3d print files, BOM, and other stuff
Connections:
- no-connect marks 23 -> 24
Other:
- note added: "ESP32 S3 supermini"
Changed lines of the file:
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@@
 		)
 	)
-	(text "MCP23017 I²C\n"
+	(text "ESP32 S3 supermini"
 		(exclude_from_sim no)
-		(at 58.928 108.966 0)
+		(at 66.04 109.982 0)
 		(effects
 			(font
@@
 	)
 	(no_connect
+		(at 52.07 139.7)
+	)
+	(no_connect
